File: MegaAmp.kicad_sch (KiCad schematic)
At the start: 28 parts, among them U1 TL972IDR

Commit message: updated silkscreen for OSHW
Other:
- title: Genesis Single Bypass Model 3 -> Genesis Model 3 Stereo Audio
Changed lines of the file:
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@@
   (paper "A")
   (title_block
-    (title "Genesis Single Bypass Model 3")
+    (title "Genesis Model 3 Stereo Audio")
     (date "2021-01-17")
     (rev "A")
     (company "Late to the Game")
-    (comment 1 "https://github.com/LateToTheGame16/sega-triple-bypass")
+    (comment 1 "https://github.com/LateToTheGame16/Genesis-Model3-Stereo")
     (comment 2 "Licensed under CERN OHL v.1.2")
     (comment 3 "For Genesis 3 consoles only")

Commit message: Saved in KiCad 8.0, fixed part descriptions
Component descriptions were wrong. Parts said 0603 but were really a 0402 footprint. No real changes to schematic or pcb. Saving from KiCad 6 to KiCad 8 created lots of format changes.
Parts:
- C1, C12, C2: Digikey 399-4925-1-ND -> (none)
- C10, C11: Digikey 399-1063-2-ND -> (none)
- C13: Digikey 445-5666-1-ND -> (none)
- C14, C15: Digikey 478-13127-1-ND -> (none)
- C5, C6, C8, C9: Digikey 1276-1184-1-ND -> (none)
- R10, R19, R20, R9: Digikey P210KHCT-ND -> (none)
- R12, R17: Digikey P130KHCT-ND -> (none)
- R15: Digikey P2.20KHCT-ND -> (none)
- R21, R22: Digikey P300KHCT-ND -> (none)
- R23, R24: Digikey P10.0KHCT-ND -> (none)
- R25, R26: Digikey P330HCT-ND -> (none)
- R5, R6: Digikey P75.0HCT-ND -> (none)
- U1: Digikey 296-22842-1-ND -> (none)
